File: robot_board/blancing_board/blancing_board.kicad_sch (KiCad schematic)
At the start: 16 parts, among them J1 POWER_SOCKET, J10 MPU6050, J2 Conn_01x13_Socket, J5 MOTORDRIVER, J6 MOTORDRIVER, J9 Conn_01x04_Socket, Q1 2SA1015, Q2 2N5551, Q3 2N5551, SW1 SW_Push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

Commit message: new page
Connections:
- net +5V: no longer U1.5 (~{LDAC}), U2.5 (~{LDAC})
- net GND: now also U1.5 (~{LDAC}), U2.5 (~{LDAC})
Changed lines of the file:
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@@
 	)
 	(junction
-		(at 123.19 50.8)
+		(at 123.19 76.2)
 		(diameter 0)
 		(color 0 0 0 0)
@@
 	)
 	(junction
-		(at 123.19 101.6)
+		(at 100.33 76.2)
 		(diameter 0)
 		(color 0 0 0 0)
@@
 	(wire
 		(pts
-			(xy 123.19 101.6) (xy 109.22 101.6)
-		)
-		(stroke
-			(width 0)
-			(type default)
-		)
-	)
-	(wire
-		(pts
 			(xy 72.39 68.58) (xy 62.23 68.58)
 		)
@@
 	(wire
 		(pts
+			(xy 100.33 76.2) (xy 123.19 76.2)
+		)
+		(stroke
+			(width 0)
+			(type default)
+		)
+	)
+	(wire
+		(pts
+			(xy 100.33 60.96) (xy 100.33 76.2)
+		)
+		(stroke
+			(width 0)
+			(type default)
+		)
+	)
+	(wire
+		(pts
+			(xy 123.19 76.2) (xy 151.13 76.2)
+		)
+		(stroke
+			(width 0)
+			(type default)
+		)
+	)
+	(wire
+		(pts
 			(xy 231.14 105.41) (xy 231.14 113.03)
 		)
@@
 	(wire
 		(pts
-			(xy 123.19 50.8) (xy 109.22 50.8)
-		)
-		(stroke
-			(width 0)
-			(type default)
-		)
-	)
-	(wire
-		(pts
 			(xy 231.14 69.85) (xy 231.14 54.61)
 		)
@@
 	(wire
 		(pts
-			(xy 151.13 76.2) (xy 123.19 76.2)
-		)
-		(stroke
-			(width 0)
-			(type default)
-		)
-	)
-	(wire
-		(pts
 			(xy 219.71 124.46) (xy 223.52 124.46)
 		)
@@
 	(wire
 		(pts
+			(xy 100.33 111.76) (xy 113.03 111.76)
+		)
+		(stroke
+			(width 0)
+			(type default)
+		)
+	)
+	(wire
+		(pts
 			(xy 128.27 162.56) (xy 138.43 162.56)
 		)
@@
 	(wire
 		(pts
-			(xy 109.22 101.6) (xy 109.22 111.76)
-		)
-		(stroke
-			(width 0)
-			(type default)
-		)
-	)
-	(wire
-		(pts
 			(xy 69.85 144.78) (xy 69.85 137.16)
 		)
@@
 	(wire
 		(pts
-			(xy 109.22 111.76) (xy 113.03 111.76)
-		)
-		(stroke
-			(width 0)
-			(type default)
-		)
-	)
-	(wire
-		(pts
 			(xy 151.13 134.62) (xy 151.13 127)
 		)
@@
 	(wire
 		(pts
-			(xy 109.22 50.8) (xy 109.22 60.96)
-		)
-		(stroke
-			(width 0)
-			(type default)
-		)
-	)
-	(wire
-		(pts
 			(xy 134.62 180.34) (xy 134.62 184.15)
 		)
@@
 	(wire
 		(pts
+			(xy 100.33 76.2) (xy 100.33 111.76)
+		)
+		(stroke
+			(width 0)
+			(type default)
+		)
+	)
+	(wire
+		(pts
 			(xy 62.23 81.28) (xy 78.74 81.28)
 		)
@@
 	(wire
 		(pts
-			(xy 109.22 60.96) (xy 113.03 60.96)
-		)
-		(stroke
+			(xy 100.33 60.96) (xy 113.03 60.96)
+		)
+		(stroke
